File: Board Files/KiCad/RP2040GPSTracker.kicad_sch (KiCad schematic)
At the start: 112 parts, among them J1 BOOTSEL, J10 GNSS_ANT, J2 RESET, J3 DEBUG, J4 BT_ANT, J5 GSM_ANT, J6 USBC_CHARGE, J7 USBC_PROG, J8 2822541-1, J9 BATTERY, U1 W25Q128JVS, U10 LM66200DRLR, U2 SIM868, U3 RP2040, U4 SN74LVC1G66DRYR, U5 LM66200DRLR, U6 MP2624GL, U7 NCP1117LPST33T3G, U8 SAFFB1G56KB0F5F, Y1 Crystal

Commit message: Rev 1.2, Swapped out C13 Footprint for more suitable one
Parts:
- C13: footprint Capacitor_Tantalum_SMD:CP_EIA-2012-15_AVX-P_Pad1.30x1.05mm_HandSolder -> Capacitor_Tantalum_SMD:CP_EIA-3528-15_AVX-H
Changed lines of the file:
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@@
     (property "Reference" "C13" (id 0) (at 292.6842 75.565 90))
     (property "Value" "100uF" (id 1) (at 294.9956 75.565 90))
-    (property "Footprint" "Capacitor_Tantalum_SMD:CP_EIA-2012-15_AVX-P_Pad1.30x1.05mm_HandSolder" (id 2) (at 300.0502 79.375 0)
+    (property "Footprint" "Capacitor_Tantalum_SMD:CP_EIA-3528-15_AVX-H" (id 2) (at 300.0502 79.375 0)
       (effects (font (size 1.27 1.27)) hide)
     )
@@
     )
     (path "/00000000-0000-0000-0000-0000627ec6f3"
-      (reference "C13") (unit 1) (value "100uF") (footprint "Capacitor_Tantalum_SMD:CP_EIA-2012-15_AVX-P_Pad1.30x1.05mm_HandSolder")
+      (reference "C13") (unit 1) (value "100uF") (footprint "Capacitor_Tantalum_SMD:CP_EIA-3528-15_AVX-H")
     )
     (path "/00000000-0000-0000-0000-0000627ec489"

Commit message: Rev 1.3. Implemented USB-C CC Channels. Fixed Z1 rotation. Expanded GPIO
Parts:
- added D7, D8: LED, LED_SMD:LED_0805_2012Metric, symbol Device:LED
- added J11: GPIO9-15, Connector_PinHeader_2.54mm:PinHeader_1x08_P2.54mm_Vertical, symbol Connector:Conn_01x08_Female
- added NT2, NT3: NetTie_2, NetTie:NetTie-2_SMD_Pad0.5mm, symbol Device:NetTie_2
- added R36, R39, R40, R41: 5.6k, Resistor_SMD:R_0603_1608Metric, symbol Device:R
- added R42, R43: 330, Resistor_SMD:R_0603_1608Metric, symbol Device:R
- C1, C10, C11, C12, C14, C15, C16, C17, C18, C19, C2, C20, C21, C22, C23, C24, C26, C27, C28, C29, C3, C30, C32, C35, C36, C37, C4, C44, C45, C5, C6, C7, C8, C9: footprint Capacitor_SMD:C_0603_1608Metric_Pad1.08x0.95mm_HandSolder -> Capacitor_SMD:C_0603_1608Metric
- C31, C34, C38, C46: footprint Capacitor_SMD:C_1206_3216Metric_Pad1.33x1.80mm_HandSolder -> Capacitor_SMD:C_1206_3216Metric
- C33: footprint Capacitor_SMD:C_0805_2012Metric_Pad1.18x1.45mm_HandSolder -> Capacitor_SMD:C_0805_2012Metric
- CR1: footprint Package_TO_SOT_SMD:SOT-363_SC-70-6_Handsoldering -> Package_TO_SOT_SMD:SOT-363_SC-70-6
- D1: footprint Diode_SMD:D_0603_1608Metric_Pad1.05x0.95mm_HandSolder -> Diode_SMD:D_0603_1608Metric
- D2, D3, D4, D5, D6: footprint LED_SMD:LED_0805_2012Metric_Pad1.15x1.40mm_HandSolder -> LED_SMD:LED_0805_2012Metric
- R1, R10, R11, R12, R13, R14, R15, R16, R17, R18, R19, R2, R20, R21, R22, R23, R24, R25, R26, R27, R28, R29, R3, R30, R31, R32, R33, R34, R35, R37, R38, R4, R5, R6, R7, R8, R9, TH1: footprint Resistor_SMD:R_0603_1608Metric_Pad0.98x0.95mm_HandSolder -> Resistor_SMD:R_0603_1608Metric
Connections:
- net BCM_D+: now also J6.B6 (D+)
- net BCM_D-: now also J6.B7 (D-)
- net GND: now also Z1.A, D7.1 (K), D8.1 (K), J11.1 (Pin_1), NT2.1, NT3.1, R36.1, R39.1, R40.1, R41.1; no longer Z1.K
- net GNDPWR: now also NT2.2, NT3.2
- net SIM_PWR: now also Z1.K; no longer Z1.A
- net USB_D+: now also J7.B6 (D+)
- net USB_D-: now also J7.B7 (D-)
- net IO_1: now reaches U3.12 (GPIO9)
- net IO_1: now also J11.2 (Pin_2)
- net IO_2: now reaches U3.13 (GPIO10)
- net IO_2: now also J11.3 (Pin_3)
- net IO_3: now reaches U3.14 (GPIO11)
- net IO_3: now also J11.4 (Pin_4)
- net IO_4: now reaches U3.15 (GPIO12)
- net IO_4: now also J11.5 (Pin_5)
- net IO_5: now reaches U3.16 (GPIO13)
- net IO_5: now also J11.6 (Pin_6)
- net IO_6: now reaches U3.17 (GPIO14)
- net IO_6: now also J11.7 (Pin_7)
- net IO_7: now reaches U3.18 (GPIO15)
- net IO_7: now also J11.8 (Pin_8)
- net at U3.27 (GPIO16): now also R42.2
- net at U3.28 (GPIO17): now also R43.2
- net at J6.A5 (CC1): now also R40.2
- net at J6.B5 (CC2): now also R41.2
- net at J7.A5 (CC1): now also R36.2
- net at J7.B5 (CC2): now also R39.2
- new net: D8.2 (A), R43.1
- new net: D7.2 (A), R42.1
- no-connect marks 58 -> 41
Other:
- moved on the sheet: C1, C10, C11, C12, C13, C14, C15, C16, C17, C18, C19, C2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

Commit message: Rev 2.0
Parts:
- added D10, D11, D9: BLUE, LED_SMD:LED_0805_2012Metric, symbol Device:LED
- added Q1, Q2: Si2319CDS, Package_TO_SOT_SMD:SOT-23, symbol Transistor_FET:Si2319CDS
- added R44: 20, Resistor_SMD:R_0603_1608Metric, symbol Device:R
- added R45: 100, Resistor_SMD:R_0603_1608Metric, symbol Device:R
- added R46: 47k, Resistor_SMD:R_0603_1608Metric, symbol Device:R
- added R47: 4.7k, Resistor_SMD:R_0603_1608Metric, symbol Device:R
- added R48: 56, Resistor_SMD:R_0603_1608Metric, symbol Device:R
- added R49: DNF, Resistor_SMD:R_0402_1005Metric, symbol Device:R
- added TP1, TP2, TP3, TP4, TP5, TP6, TP7, TP8, TP9: TestPoint, TestPoint:TestPoint_Pad_1.5x1.5mm, symbol Connector:TestPoint
- C1, C10, C11, C12, C2, C3, C4, C5, C6, C7, C8, C9: footprint Capacitor_SMD:C_0603_1608Metric -> Capacitor_SMD:C_0402_1005Metric
- D3, D7, D8: value LED -> RED
- D4, D5, D6: value LED -> BLUE
- J1, J2: footprint Button_Switch_SMD:TS-1145A-C-A -> Button_Switch_SMD:SW_SPST_ALPS_SKRKAEE020
- J10: value GNSS_ANT -> GNSS
- J11: footprint Connector_PinHeader_2.54mm:PinHeader_1x08_P2.54mm_Vertical -> Connector_PinHeader_2.54mm:PinHeader_1x09_P2.54mm_Vertical; symbol Connector:Conn_01x08_Female -> Connector:Conn_01x09_Female
- J4: value BT_ANT -> BT(LE)
- J5: value GSM_ANT -> GSM
- R22, R42, R43: value 330 -> 56
- R23, R30, R31: value 330 -> 20
- R28: value 1k -> 100/0.2
- R36, R39, R40, R41: value 5.6k -> 5.1k; footprint Resistor_SMD:R_0603_1608Metric -> Resistor_SMD:R_0402_1005Metric
- U1: footprint Package_SO:SOIC-8_5.23x5.23mm_P1.27mm -> Package_SON:WSON-8-1EP_6x5mm_P1.27mm_EP3.4x4.3mm
- Y1: footprint Crystal:Crystal_SMD_HC49-SD -> ABRACON:ABMM2-12.000MHZ-E2-T; symbol Device:Crystal -> ABRACON:ABMM2-12.000MHZ-E2-T
Connections:
- net +1V1: now also TP3.1
- net +3V3: now also J11.9 (Pin_9), Q1.2 (S), R49.1, TP4.1
- net BOOST_OUT: now also TP8.1
- net GND: now also U1.9 (PAD), Y1.2 (GND), Y1.4 (GND), D10.1 (K), D9.1 (K), Q2.3 (D), R46.2; no longer J10.4 (GND), J4.4 (GND), J5.4 (GND)
- net GNDPWR: now also TP9.1
- net SIM_C_DET: now also CR1.4; no longer CR1.6
- net SIM_C_VDD: now also CR1.3; no longer CR1.1
- net SIM_PWR: now also D11.2 (A), TP5.1
- net USB_BOOT: now also TP7.1
- net USB_D+: now also TP2.1
- net USB_D-: now also TP1.1
- net PI_RESET: now reaches J2.1 (A), U3.26 (RUN)
- net PI_RESET: now also TP6.1
- net LED_1: now reaches R42.2, U3.27 (GPIO16)
- net LED_2: now reaches R43.2, U3.28 (GPIO17)
- net LED_3: now reaches R22.2, U3.29 (GPIO18)
- net LED_4: now reaches R23.2, U3.30 (GPIO19)
- net LED_5: now reaches R30.2, U3.31 (GPIO20)
- net LED_6: now reaches R31.2, U3.32 (GPIO21)
- net LED_7: now reaches U3.36 (GPIO24)
- net LED_7: now also R44.2
- net LED_PWR: now reaches U3.37 (GPIO25)
- net LED_PWR: now also Q1.1 (G)
- net PI_D-: now reaches R2.2, U3.46 (USB_DM)
- net PI_D+: now reaches R1.2, U3.47 (USB_DP)
- net SPI_IO3: now reaches U1.7 (IO3), U3.51 (QSPI_SD3)
- net SPI_CLK: now reaches U1.6 (CLK), U3.52 (QSPI_SCLK)
- net SPI_IO0: now reaches U1.5 (DI(IO0)), U3.53 (QSPI_SD0)
- net SPI_IO2: now reaches U1.3 (IO2), U3.54 (QSPI_SD2)
- net SPI_IO1: now reaches U1.2 (DO(IO1)), U3.55 (QSPI_SD1)
- net SPI_SS: now reaches R5.1, U1.1 (~{CS}), U3.56 (QSPI_SS)
- net SPI_SS: now also R49.2
- net at C20.1, R17.2: now also Y1.3; no longer Y1.2
- net SIM_NETLIGHT: now reaches U2.41 (NETLIGHT)
- net SIM_NETLIGHT: now also R47.1
- net at C28.2, J8.2 (C2), R24.1: now also CR1.5; no longer CR1.3
- net at C29.2, J8.3 (C3), R25.1: now also CR1.6; no longer CR1.4
- net at C30.2, J8.6 (C7), R26.1: now also CR1.1; no longer CR1.5
- new net: Q1.3 (D), R45.2
- new net: D10.2 (A), R45.1
- new net: D9.2 (A), R44.1
- new net: Q2.1 (G), R46.1, R47.2
- new net: Q2.2 (S), R48.1
- new net: D11.1 (K), R48.2
- no-connect marks 41 -> 39
Other:
- moved on the sheet: C19, C20, D3, D4, D5, D6, D7, D8, R22, R23, R30, R31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

Commit message: Rev 3.1 - Power-stage overhaul, SIM power finetuning
Parts:
- removed U4: SN74LVC1G66DRYR, TI_LV74XXG6:SN74LVC1G66DRYR, symbol TI_SN74XXG66:SN74LVC1G66DRYR
- removed U7: NCP1117LPST33T3G, Package_TO_SOT_SMD:SOT-223, symbol NCP1117:NCP1117LPST33T3G
- added C25: 22pF, Capacitor_SMD:C_0603_1608Metric, symbol Device:C
- added C39: 22nF, Capacitor_SMD:C_0603_1608Metric, symbol Device:C
- added C40, C41: 22uF, Capacitor_SMD:C_0603_1608Metric, symbol Device:C
- added C42: 10uF, Capacitor_SMD:C_0603_1608Metric, symbol Device:C
- added L1: 1uH, Inductor_SMD:L_1008_2520Metric, symbol Device:L
- added L3: 4.7uH, Inductor_SMD:MCS-0530, symbol Device:L
- added R50, R52, R53: 100k, Resistor_SMD:R_0603_1608Metric, symbol Device:R
- added R51: 22k, Resistor_SMD:R_0603_1608Metric, symbol Device:R
- added R54: 17.1k, Resistor_SMD:R_0603_1608Metric, symbol Device:R
- added U4: RT8096, Package_TO_SOT_SMD:TSOT-23-5, symbol Converter_DCDC:RT8096
- added U7: SD8942, Package_TO_SOT_SMD:SOT-23-6, symbol Converter_DCDC:SD8942
- J9: footprint Connector_JST:JST_PH_B2B-PH-K_1x02_P2.00mm_Vertical -> Connector_JST:JST_PH_S2B-PH-K_1x02_P2.00mm_Horizontal
Connections:
- net +3V3: now also C37.1, C25.1, L1.2, R50.1; no longer C37.2
- net GND: now also C37.2, C40.2, C41.2, C42.1, R51.2, R54.2, U4.2 (GND), U7.2 (GND); no longer C37.1
- net PI_VREG_IN: now also U4.1 (EN), U4.4 (VIN)
- net PROG_VBUS: now also C42.2, R53.1, U7.5 (IN); no longer U5.3 (VIN1)
- new net: R52.2, R54.1, U7.3 (FB)
- new net: R53.2, U7.4 (EN)
- new net PI_VREG_FB: C25.2, R50.2, R51.1, U4.5 (FB)
- new net PI_VREG_SW: L1.1, U4.3 (SW)
- new net SIM_VREG_BTS: C39.1, U7.1 (BS)
- new net SIM_VREG_OUT: C39.2, C40.1, C41.1, L3.1, L3.2, R52.1, U5.3 (VIN1), U7.6 (SW)
- no-connect marks 39 -> 38
Other:
- note removed: "BCM Disable on prog-mode"
- moved on the sheet: C35, C37
